File: logicbone.kicad_pcb (KiCad board)
At the start: 6 copper layers, 86.4 x 54.6 mm, 267 parts, among them IC1 ECP5UM-CABGA554, IC10 AT25SF081-XMHF-X, IC11 FAN53600AUC33X, IC12 74LVC1G07, IC13 TPS51200, IC14 KSZ9031RNXCA, IC2 DDR3-TFBGA96, IC3 DDR3-TFBGA96, IC4 ACT8846QM460, IC5 PI6CG18401, IC6 74LVC1G02, IC8 STM32FLxx-QFN48, IC9 ADC120, J1 NGFF-KEY-E, J2 GCT_USB4110_USBC, J3 ARJM11xx-502, J4 FTSH-105-DV-K, J6 Micro_SD_MEM2075, P8 BB_2x23, P9 BB_2x23, SW1 SW_SPST, SW2 SW_SPST, Y1 25MHz, Y2 32.768kHz

Commit message: Revert back to a 16-bit DDR3 bus, initial DDR3 layout.
The caBGA-554 package was too large and fat to reasonably be able
to fit within the beaglebone footprint and still leave enough room
for DDR3 and the expansion headers. So, it seems more sensible to
switch back to a 16-bit wide bus.

Now that we can fit everything, take a first stab at getting the DDR3
data busses routed and length matched.
Parts:
- removed C200, C243, C244: 100nF, Capacitor_SMD:C_0402_1005Metric
- removed C510, C511: 10nF, Capacitor_SMD:C_0402_1005Metric
- removed R11, R12, R9: 50, Resistor_SMD:R_0402_1005Metric
- removed R26: R, Resistor_SMD:R_0402_1005Metric
- removed REF**: MountingHole_3.2mm_M3, MountingHole:MountingHole_3.2mm_M3
- removed REF**: USB4110, Logicbone:USB4110
- C252, C253, C254, C257, C258, C259: footprint Capacitor_SMD:C_0603_1608Metric -> Capacitor_SMD:C_0402_1005Metric; moved to B.Cu
- C281, C515, C516, C517, C520, C521, C525, C527: moved to B.Cu
- C505: value 100nF -> 10nF
- IC1: value ECP5UM-CABGA554 -> ECP5UM-CABGA381; footprint Logicbone:caBGA-554_26x26_23.0x23.0mm -> Logicbone:caBGA-381_20x20_17.0x17.0mm
- IC2, IC3: value DDR3-TFBGA96 -> DDR3-TFBGA78; footprint Logicbone:FBGA-96_10.0x14.0mm_DDR3L_P0.8mm -> Package_BGA:FBGA-78_7.5x11mm_Layout2x3x13_P0.8mm
- R7: value 50 -> R_Small
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Connections:
- C210 pad 1: VCCIOA -> VCC
- C211 pad 1: VCCIOA -> VCC
- C212 pad 1: VCCIOA -> VCC
- C220 pad 1: VCC -> VCCIOA
- C221 pad 1: VCC -> VCCIOA
- C222 pad 1: VCC -> VCCIOA
- IC1 pad A10: Net-(IC1-PadA10) -> /Exp Headers/ADC_SCLK
- IC1 pad A11: Net-(IC1-PadA11) -> /Exp Headers/ADC_MISO
- IC1 pad A14: /Exp Headers/P8_LVDS5p -> /Ethernet/MMC_CLK
- IC1 pad A15: /Exp Headers/P8_LVDS5n -> /Ethernet/MDIO_DATA
- IC1 pad A16: /Exp Headers/P8_LVDS8p -> /Ethernet/ETH_TXD0
- IC1 pad A17: /Exp Headers/P8_LVDS8n -> /Ethernet/ETH_RXD2
- IC1 pad A18: /Exp Headers/P8_LVDS14p -> /Ethernet/ETH_TXCLK
- IC1 pad A19: /Exp Headers/P8_LVDS14n -> /Ethernet/ETH_RXCLK
- IC1 pad A2: /Exp Headers/P9_GPIO11 -> /FPGA Memory/DDR3_DQ10
- IC1 pad A3: /Exp Headers/P9_GPIO12 -> Net-(IC1-PadA3)
- IC1 pad A4: /Exp Headers/P9_GPIO14 -> Net-(IC1-PadA4)
- IC1 pad A5: /Exp Headers/P9_GPIO23 -> Net-(IC1-PadA5)
- IC1 pad A6: /Exp Headers/P9_GPIO24 -> /Exp Headers/P9_GPIO11
- IC1 pad A8: /Exp Headers/P9_GPIO25 -> /Exp Headers/P9_GPIO26
- IC1 pad A9: /Exp Headers/P9_GPIO26 -> /Exp Headers/P9_CLKOUT
- IC1 pad B1: /FPGA Memory/DDR3_DQ6 -> /FPGA Memory/DDR3_DQ8
- IC1 pad B10: /Exp Headers/ADC_MOSI -> /Exp Headers/~ADC_CSEL
- IC1 pad B11: Net-(IC1-PadB11) -> /Exp Headers/ADC_MOSI
- IC1 pad B12: GND -> /Ethernet/LED_USER3
- IC1 pad B13: /Exp Headers/P8_LVDS4p -> Net-(IC1-PadB13)
- IC1 pad B14: /Exp Headers/P8_LVDS4n -> GND
- IC1 pad B15: GND -> /Ethernet/MDIO_CLK
- IC1 pad B16: /Exp Headers/P8_LVDS7p -> /Ethernet/ETH_TXD1
- IC1 pad B17: /Exp Headers/P8_LVDS9p -> /Ethernet/ETH_RXD0
- IC1 pad B18: GND -> /Ethernet/ETH_RXD3
- IC1 pad B19: /Exp Headers/P8_LVDS13n -> /Ethernet/ETH_RXCTL
- IC1 pad B2: GND -> /FPGA Memory/DDR3_VREF
- IC1 pad B3: /FPGA Memory/DDR3_DQ7 -> /FPGA Memory/DDR3_A4
- IC1 pad B4: /Exp Headers/P9_GPIO13 -> /FPGA Memory/DDR3_A11
- IC1 pad B5: GND -> /FPGA Memory/DDR3_A6
- IC1 pad B6: /Exp Headers/P9_GPIO22 -> /Exp Headers/P9_GPIO12
- IC1 pad B8: /Exp Headers/P9_GPIO27 -> /Exp Headers/P9_GPIO24
- IC1 pad B9: GND -> /Exp Headers/P9_SPI_D0
- IC1 pad C1: /FPGA Memory/DDR3_DQ1 -> /FPGA Memory/DDR3_DQ14
- IC1 pad C10: /Exp Headers/ADC_MISO -> Net-(IC1-PadC10)
- IC1 pad C11: /Exp Headers/P9_CLKOUT -> Net-(IC1-PadC11)
- IC1 pad C12: Net-(IC1-PadC12) -> /Ethernet/LED_USER4
- IC1 pad C13: /Exp Headers/P8_LVDS3p -> /Ethernet/MMC_DAT2
- IC1 pad C14: /Exp Headers/P8_LVDS3n -> /Ethernet/MMC_DAT0
- IC1 pad C15: Net-(IC1-PadC15) -> /Ethernet/~ETH_RESET
- IC1 pad C16: /Exp Headers/P8_LVDS7n -> /Ethernet/ETH_TXD2
- IC1 pad C17: /Exp Headers/P8_LVDS9n -> /Ethernet/ETH_RXD1
- IC1 pad C18: /Exp Headers/P8_LVDS11p -> /Exp Headers/P8_LVDS1p
- IC1 pad C19: /Exp Headers/P8_LVDS13p -> GND
- IC1 pad C2: /FPGA Memory/DDR3_DQ0 -> /FPGA Memory/DDR3_DQ12
- IC1 pad C3: /FPGA Memory/DDR3_DQ3 -> /FPGA Memory/DDR3_A12
- IC1 pad C4: /FPGA Memory/DDR3_DQ2 -> /FPGA Memory/DDR3_A1
- IC1 pad C5: /Exp Headers/P9_GPIO16 -> /FPGA Memory/DDR3_A8
- IC1 pad C6: /Exp Headers/P9_GPIO21 -> /Exp Headers/P9_GPIO17
- IC1 pad C8: /Exp Headers/P9_GPIO42 -> /Exp Headers/P9_GPIO23
- IC1 pad C9: /Exp Headers/P9_SPI_D0 -> /Exp Headers/~P9_SPI_CSEL
- IC1 pad D1: /FPGA Memory/~DDR3_CAS -> /FPGA Memory/DDR3_DQ13
- IC1 pad D10: /Exp Headers/ADC_SCLK -> /Exp Headers/P9_SPI_SCLK
- IC1 pad D11: Net-(IC1-PadD11) -> /Ethernet/LED_USER1
- IC1 pad D12: Net-(IC1-PadD12) -> /Ethernet/ETH_REFCLK
- IC1 pad D13: /Exp Headers/P8_LVDS2p -> /Ethernet/MMC_DAT3
- IC1 pad D14: /Exp Headers/P8_LVDS2n -> /Ethernet/MMC_DAT1
- IC1 pad D15: Net-(IC1-PadD15) -> /Ethernet/~ETH_INT
- IC1 pad D16: /Exp Headers/P8_LVDS6p -> /Ethernet/ETH_TXD3
- IC1 pad D17: /Exp Headers/P8_LVDS10p -> /Exp Headers/P8_LVDS1n
- IC1 pad D18: /Exp Headers/P8_LVDS11n -> /Exp Headers/P8_LVDS3p
- IC1 pad D19: /Exp Headers/P8_LVDS12n -> /Exp Headers/P8_LVDS9n
- IC1 pad D2: /FPGA Memory/DDR3_DQS0+ -> Net-(IC1-PadD2)
- IC1 pad D3: /FPGA Memory/DDR3_DQ5 -> Net-(IC1-PadD3)
- IC1 pad D4: /FPGA Memory/DDR3_DQ4 -> GND
- IC1 pad D5: /Exp Headers/P9_GPIO15 -> /FPGA Memory/DDR3_A10
- IC1 pad D6: /Exp Headers/P9_GPIO18 -> /Exp Headers/P9_GPIO14
- IC1 pad D8: /Exp Headers/P9_SPI_SCLK -> /Exp Headers/P9_GPIO22
- IC1 pad D9: /Exp Headers/P9_SPI_D1 -> /Exp Headers/P9_GPIO27
- IC1 pad E1: /FPGA Memory/DDR3_DQS0- -> /FPGA Memory/DDR3_DQ11
- IC1 pad E10: /Exp Headers/~ADC_CSEL -> /Exp Headers/P9_SPI_D1
- IC1 pad E11: Net-(IC1-PadE11) -> /Ethernet/LED_USER2
- IC1 pad E12: GND -> Net-(IC1-PadE12)
- IC1 pad E13: /Exp Headers/P8_LVDS1p -> /Ethernet/MMC_CMD
- IC1 pad E14: /Exp Headers/P8_LVDS1n -> /Ethernet/MMC_DET
- IC1 pad E15: GND -> Net-(IC1-PadE15)
- IC1 pad E16: /Exp Headers/P8_LVDS6n -> /Exp Headers/P8_LVDS2p
- IC1 pad E17: /Exp Headers/P8_LVDS10n -> /Exp Headers/P8_LVDS3n
- IC1 pad E18: GND -> /Exp Headers/P8_LVDS4p
- IC1 pad E19: /Exp Headers/P8_LVDS12p -> /Exp Headers/P8_LVDS10n
- IC1 pad E2: GND -> /FPGA Memory/DDR3_DQ15
- IC1 pad E3: /FPGA Memory/~DDR3_RAS -> /FPGA Memory/DDR3_A9
- IC1 pad E4: /FPGA Memory/~DDR3_CS -> /FPGA Memory/DDR3_A7
- IC1 pad E5: GND -> /FPGA Memory/DDR3_A2
- IC1 pad E6: /Exp Headers/P9_GPIO17 -> /Exp Headers/P9_GPIO13
- IC1 pad E8: /Exp Headers/~P9_SPI_CSEL -> /Exp Headers/P9_GPIO21
- IC1 pad E9: GND -> /Exp Headers/P9_GPIO42
- IC1 pad F1: /FPGA Memory/DDR3_DM1 -> /FPGA Memory/DDR3_DQ6
- IC1 pad F10: Net-(IC1-PadF10) -> VCC
- IC1 pad F12: Net-(IC1-PadF12) -> VCC
- IC1 pad F13: Net-(IC1-PadF13) -> GND
- IC1 pad F14: Net-(IC1-PadF14) -> GND
- IC1 pad F15: Net-(IC1-PadF15) -> VCCAUX
- IC1 pad F17: Net-(IC1-PadF17) -> /Exp Headers/P8_LVDS5p
- IC1 pad F18: Net-(IC1-PadF18) -> /Exp Headers/P8_LVDS4n
- IC1 pad F19: Net-(IC1-PadF19) -> /Exp Headers/P8_LVDS11n
- IC1 pad F2: /FPGA Memory/DDR3_DM0 -> Net-(IC1-PadF2)
- IC1 pad F3: /FPGA Memory/~DDR3_WE -> /FPGA Memory/DDR3_DQ9
- IC1 pad F4: /FPGA Memory/DDR3_DQ9 -> /FPGA Memory/DDR3_A5
- IC1 pad F5: /FPGA Memory/DDR3_DQ8 -> /FPGA Memory/DDR3_A3
- IC1 pad F8: Net-(IC1-PadF8) -> GND
- IC1 pad F9: Net-(IC1-PadF9) -> VCC
- IC1 pad H1: /FPGA Memory/DDR3_ODT1 -> /FPGA Memory/DDR3_DQ7
- IC1 pad H10: VCC -> VCORE
- IC1 pad H11: VCCAUX -> VCORE
- IC1 pad H12: VCC -> VCORE
- IC1 pad H13: VCC -> VCORE
- IC1 pad H14: VCCAUX -> VCCIOA
- IC1 pad H16: VCCIOA -> /Exp Headers/P8_LVDS6n
- IC1 pad H17: VCCAUX -> /Exp Headers/P8_LVDS7n
- IC1 pad H18: VCCIOA -> /Exp Headers/P8_LVDS7p
- IC1 pad H2: /FPGA Memory/DDR3_BA2 -> /FPGA Memory/DDR3_DQ4
- IC1 pad H3: /FPGA Memory/DDR3_BA0 -> Net-(IC1-PadH3)
- IC1 pad H4: /FPGA Memory/DDR3_DQ12 -> /FPGA Memory/DDR3_DQS1+
- IC1 pad H5: /FPGA Memory/DDR3_VREF -> /FPGA Memory/DDR3_DM1
- IC1 pad H6: /FPGA Memory/DDR3_ODT0 -> VDDR
- IC1 pad H8: GND -> VCORE
- IC1 pad H9: GND -> VCORE
- IC1 pad J1: /FPGA Memory/DDR3_DQ17 -> /FPGA Memory/DDR3_DQS0-
- IC1 pad J13: GND -> VCORE
- IC1 pad J15: GND -> VCCIOA
- IC1 pad J16: GND -> /Exp Headers/P8_LVDS8n
- IC1 pad J17: GND -> /Exp Headers/P8_LVDS8p
- IC1 pad J18: GND -> /Exp Headers/P8_LVDS14p
- IC1 pad J19: VCC -> /Exp Headers/P8_LVDS15p
- IC1 pad J3: /FPGA Memory/DDR3_BA1 -> /FPGA Memory/DDR3_DQ5
- IC1 pad J4: /FPGA Memory/DDR3_DQS1- -> /FPGA Memory/DDR3_DM0
- IC1 pad J5: GND -> Net-(IC1-PadJ5)
- IC1 pad J6: /FPGA Memory/DDR3_DQ10 -> VDDR
- IC1 pad J8: GND -> VCORE
- IC1 pad K1: /FPGA Memory/DDR3_DQ20 -> /FPGA Memory/DDR3_DQ1
- IC1 pad K11: VCORE -> GND
- IC1 pad K12: VCORE -> GND
- IC1 pad K14: VCORE -> GND
- IC1 pad K15: VCORE -> GND
- IC1 pad K16: VCORE -> Net-(IC1-PadK16)
- IC1 pad K17: GND -> Net-(IC1-PadK17)
- IC1 pad K18: GND -> /Exp Headers/P8_LVDS14n
- IC1 pad K19: VCCAUX -> /Exp Headers/P8_LVDS15n
- IC1 pad K2: /FPGA Memory/DDR3_DQ16 -> /FPGA Memory/DDR3_DQS0+
- IC1 pad K3: /FPGA Memory/DDR3_DQ18 -> /FPGA Memory/DDR3_DQ3
- IC1 pad K4: /FPGA Memory/DDR3_CK+ -> /FPGA Memory/~DDR3_CS
- IC1 pad K5: /FPGA Memory/DDR3_DQS1+ -> /FPGA Memory/DDR3_VREF
- IC1 pad K6: /FPGA Memory/DDR3_DQ11 -> GND
- IC1 pad K8: VDDR -> VCORE
- IC1 pad L1: /FPGA Memory/DDR3_DQ21 -> /FPGA Memory/~DDR3_CAS
- IC1 pad L10: VCORE -> GND
- IC1 pad L13: GND -> VCORE
- IC1 pad L14: GND -> VCCIOB
- IC1 pad L15: GND -> VCCIOB
- IC1 pad L16: GND -> /FPGA SERDES/M2_SDIO_DATA2
- IC1 pad L17: VCORE -> /FPGA SERDES/M2_SDIO_DATA3
- IC1 pad L18: GND -> /FPGA SERDES/~M2_SDIO_WAKE
- IC1 pad L19: VCC -> /FPGA SERDES/M2_SDIO_DATA0
- IC1 pad L2: /FPGA Memory/DDR3_DQS2+ -> /FPGA Memory/DDR3_ODT0
- IC1 pad L3: /FPGA Memory/DDR3_DQ19 -> Net-(IC1-PadL3)
- IC1 pad L4: /FPGA Memory/DDR3_CK- -> Net-(IC1-PadL4)
- IC1 pad L5: /FPGA Memory/DDR3_DQ13 -> Net-(IC1-PadL5)
- IC1 pad L8: VCCAUX -> VCORE
- IC1 pad M1: /FPGA Memory/DDR3_DQS2- -> /FPGA Memory/~DDR3_WE
- IC1 pad M10: VCORE -> GND
- IC1 pad M13: GND -> VCORE
- IC1 pad M15: GND -> VCCIOB
- IC1 pad M17: VCORE -> /FPGA SERDES/M2_PCM_SYNC
- IC1 pad M18: GND -> /FPGA SERDES/~M2_SDIO_RESET
- IC1 pad M19: VCC -> /FPGA SERDES/M2_SDIO_DATA1
- IC1 pad M3: /FPGA Memory/DDR3_DQ23 -> /FPGA Memory/DDR3_BA2
- IC1 pad M4: /FPGA Memory/DDR3_DQ15 -> /FPGA Memory/DDR3_CK+
- IC1 pad M5: GND -> Net-(IC1-PadM5)
- IC1 pad M6: /FPGA Memory/DDR3_DQ14 -> VDDR
- IC1 pad M8: VDDR -> VCORE
- IC1 pad N11: GND -> VCORE
- IC1 pad N12: GND -> VCORE
- IC1 pad N13: GND -> VCORE
- IC1 pad N16: GND -> /FPGA SERDES/M2_PCM_CLK
- IC1 pad N17: VCORE -> /FPGA SERDES/M2_RTS
- IC1 pad N18: GND -> /FPGA SERDES/M2_PCM_IN
- IC1 pad N19: VCC -> /FPGA SERDES/M2_COEX1
- IC1 pad N2: /FPGA Memory/DDR3_VREF -> /FPGA Memory/DDR3_CKE
- IC1 pad N3: /FPGA Memory/DDR3_DQ22 -> /FPGA Memory/DDR3_BA1
- IC1 pad N4: /FPGA Memory/DDR3_DQ27 -> /FPGA Memory/~DDR3_RST
- IC1 pad N5: /FPGA Memory/~DDR3_RST -> /FPGA Memory/DDR3_CK-
- IC1 pad N6: /FPGA Memory/DDR3_CKE -> GND
- IC1 pad N8: VDDR -> VCORE
- IC1 pad N9: GND -> VCORE
- IC1 pad P1: /FPGA Memory/DDR3_A9 -> /FPGA Memory/~DDR3_RAS
- IC1 pad P10: VCORE -> +3V3
- IC1 pad P15: GND -> VCCAUX
- IC1 pad P16: GND -> /FPGA SERDES/M2_CTS
- IC1 pad P17: VCORE -> /FPGA SERDES/M2_PCM_OUT
- IC1 pad P18: GND -> /FPGA SERDES/~M2_RESET
- IC1 pad P19: VCCIOB -> /FPGA SERDES/M2_COEX3
- IC1 pad P2: /FPGA Memory/DDR3_A8 -> /FPGA Memory/DDR3_A0
- IC1 pad P3: /FPGA Memory/DDR3_A7 -> Net-(IC1-PadP3)
- IC1 pad P4: /FPGA Memory/DDR3_DQ24 -> Net-(IC1-PadP4)
- IC1 pad P5: /FPGA Memory/DDR3_DQ25 -> /FPGA Memory/DDR3_BA0
- IC1 pad P6: /FPGA Memory/DDR3_DQ26 -> VCCAUX
- IC1 pad P8: VDDR -> GND
- IC1 pad P9: GND -> +3V3
- IC1 pad R1: /FPGA Memory/DDR3_A11 -> /Exp Headers/SCL
- IC1 pad R16: GND -> /FPGA SERDES/M2_RXD
- IC1 pad R17: VCORE -> /FPGA SERDES/M2_TXD
- IC1 pad R18: GND -> /FPGA SERDES/M2_VEND1
- IC1 pad R19: VCCIOB -> GND
- IC1 pad R2: GND -> Net-(IC1-PadR2)
- IC1 pad R3: /FPGA Memory/DDR3_A6 -> Net-(IC1-PadR3)
- IC1 pad R4: /FPGA Memory/DDR3_DQ28 -> Net-(IC1-PadR4)
- IC1 pad R5: GND -> /Supervisor/FPGA_TDI
- IC1 pad T1: /FPGA Memory/DDR3_A15 -> /Exp Headers/SDA
- IC1 pad T10: VCORE -> /FPGA SERDES/VCCTRX0
- IC1 pad T11: VCORE -> /FPGA SERDES/VCCTRX1
- IC1 pad T12: VCORE -> /FPGA SERDES/VCCTRX1
- IC1 pad T13: VCORE -> /FPGA SERDES/VCCTRX1
- IC1 pad T14: VCORE -> /FPGA SERDES/VCCTRX1
- IC1 pad T15: VCORE -> /FPGA Power/VCCA1
- IC1 pad T16: VCORE -> Net-(IC1-PadT16)
- IC1 pad T17: VCORE -> /FPGA SERDES/FPGA_REFCLKn
- IC1 pad T18: GND -> /FPGA SERDES/~M2_ALERT
- IC1 pad T19: VCCAUX -> /FPGA SERDES/M2_VEND2
- IC1 pad T2: /FPGA Memory/DDR3_A10 -> /Supervisor/~FPGA_CSEL
- IC1 pad T3: /FPGA Memory/DDR3_A4 -> Net-(IC1-PadT3)
- IC1 pad T4: /FPGA Memory/DDR3_DQ30 -> Net-(IC1-PadR4)
- IC1 pad T5: /FPGA Memory/DDR3_DQ29 -> /Supervisor/FPGA_TCK
- IC1 pad T8: VCCAUX -> /FPGA SERDES/VCCTRX0
- IC1 pad T9: GND -> /FPGA SERDES/VCCTRX0
- IC1 pad U1: /FPGA Memory/DDR3_A14 -> Net-(IC1-PadU1)
- IC1 pad U15: GND -> /FPGA Power/VCCA1
- IC1 pad U16: GND -> /FPGA SERDES/FPGA_REFCLKp
- IC1 pad U17: GND -> /FPGA SERDES/M2_USB_DM
- IC1 pad U18: GND -> /FPGA SERDES/M2_USB_DP
- IC1 pad U19: VCCIOB -> /FPGA SERDES/M2_VEND0
- IC1 pad U2: /FPGA Memory/DDR3_A13 -> /Supervisor/~FPGA_HOLDN
- IC1 pad U3: /FPGA Memory/DDR3_A5 -> /Supervisor/FPGA_SCLK
- IC1 pad U4: /FPGA Memory/DDR3_DM3 -> Net-(IC1-PadU4)
- IC1 pad U5: /FPGA Memory/DDR3_DQS3- -> /Supervisor/FPGA_TMS
- IC1 pad U6: /FPGA Memory/DDR3_DM2 -> /FPGA Power/VCCA0
- IC1 pad U8: VDDR -> GND
- IC1 pad V1: /FPGA Memory/DDR3_A12 -> /Supervisor/FPGA_UART_CLK
- IC1 pad V10: +3V3 -> VCCAUXTRX
- IC1 pad V11: +3V3 -> VCCAUXTRX
- IC1 pad V17: GND -> VCCAUXTRX
- IC1 pad V18: VMMC -> VCCAUXTRX
- IC1 pad V19: VMMC -> GND
- IC1 pad V2: GND -> /Supervisor/FPGA_MISO
- IC1 pad V3: Net-(IC1-PadV3) -> /Supervisor/~FPGA_INIT
- IC1 pad V4: /FPGA Memory/DDR3_DQS3+ -> /Supervisor/FPGA_TDO
- IC1 pad V6: /FPGA Memory/DDR3_A1 -> GND
- IC1 pad V8: VDDR -> GND
- IC1 pad W1: Net-(IC1-PadW1) -> /Supervisor/FPGA_UART_TXD
- IC1 pad W10: /FPGA SERDES/VCCTRX0 -> Net-(IC1-PadW10)
- IC1 pad W11: /FPGA SERDES/VCCTRX0 -> Net-(IC1-PadW11)
- IC1 pad W12: /FPGA SERDES/VCCTRX0 -> GND
- IC1 pad W13: /FPGA SERDES/VCCTRX0 -> Net-(C115-Pad1)
- IC1 pad W14: /FPGA SERDES/VCCTRX1 -> Net-(C114-Pad1)
- IC1 pad W15: /FPGA SERDES/VCCTRX1 -> GND
- IC1 pad W16: /FPGA SERDES/VCCTRX1 -> GND
- IC1 pad W17: /FPGA SERDES/VCCTRX1 -> Net-(C113-Pad1)
- IC1 pad W18: GND -> Net-(C112-Pad1)
- IC1 pad W19: VCCAUX -> GND
- IC1 pad W2: Net-(IC1-PadW2) -> /Supervisor/FPGA_MOSI
- IC1 pad W3: Net-(IC1-PadW3) -> /Ethernet/~SYS_RESET
- IC1 pad W4: /FPGA Memory/DDR3_A0 -> Net-(IC1-PadW4)
- IC1 pad W5: /FPGA Memory/DDR3_A2 -> Net-(IC1-PadW5)
- IC1 pad W6: /FPGA Memory/DDR3_A3 -> GND
- IC1 pad W8: VCCAUX -> Net-(IC1-PadW8)
- IC1 pad W9: GND -> Net-(IC1-PadW9)
- IC2 pad A1: /DDR3 Power/VDDR_IO -> GND
- IC2 pad A2: /FPGA Memory/DDR3_DQ13 -> /DDR3 Power/VDDR_CORE
- IC2 pad A3: /FPGA Memory/DDR3_DQ15 -> Net-(IC2-PadA3)
- IC2 pad A7: /FPGA Memory/DDR3_DQ12 -> /FPGA Memory/DDR3_DM0
- IC2 pad A8: /DDR3 Power/VDDR_IO -> GND
- IC2 pad A9: GND -> /DDR3 Power/VDDR_CORE
- IC2 pad B2: /DDR3 Power/VDDR_CORE -> GND
- IC2 pad B3: GND -> /FPGA Memory/DDR3_DQ0
- IC2 pad B7: /FPGA Memory/DDR3_DQS1- -> Net-(IC2-PadB7)
- IC2 pad B8: /FPGA Memory/DDR3_DQ14 -> GND
- IC2 pad B9: GND -> /DDR3 Power/VDDR_IO
- IC2 pad C2: /FPGA Memory/DDR3_DQ11 -> /FPGA Memory/DDR3_DQ2
- IC2 pad C3: /FPGA Memory/DDR3_DQ9 -> /FPGA Memory/DDR3_DQS0+
- IC2 pad C7: /FPGA Memory/DDR3_DQS1+ -> /FPGA Memory/DDR3_DQ1
- IC2 pad C8: /FPGA Memory/DDR3_DQ10 -> /FPGA Memory/DDR3_DQ3
- IC2 pad C9: /DDR3 Power/VDDR_IO -> GND
- IC2 pad D2: /DDR3 Power/VDDR_IO -> /FPGA Memory/DDR3_DQ6
- IC2 pad D3: /FPGA Memory/DDR3_DM1 -> /FPGA Memory/DDR3_DQS0-
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Routing:
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- removed copper zone on In1.Cu, net GND
Other:
- copper layers 6 -> 8
- net class DDR3_CTRL added: clearance 0.08, trace_width 0.14, via_dia 0.5, via_drill 0.2
- net class DDR3_DQ added: clearance 0.08, trace_width 0.14, via_dia 0.5, via_drill 0.2
- net class DDR3_DQS added: clearance 0.08, trace_width 0.1, via_dia 0.5, via_drill 0.2

Commit message: Complete routing of the DDR interface.
This is the last of the DDR3 signals connected, but we still need to
revisit the length tuning.
Parts:
- C403: moved to B.Cu
- moved C403 260.0 mm to (140.2, 82.7)
Connections:
- IC1 pad A3: Net-(IC1-PadA3) -> /FPGA Memory/DDR3_A3
- IC1 pad A4: Net-(IC1-PadA4) -> /FPGA Memory/DDR3_A2
- IC1 pad A5: Net-(IC1-PadA5) -> /FPGA Memory/DDR3_A7
- IC1 pad B3: /FPGA Memory/DDR3_A4 -> /FPGA Memory/DDR3_A0
- IC1 pad B4: /FPGA Memory/DDR3_A11 -> /FPGA Memory/DDR3_BA0
- IC1 pad B5: /FPGA Memory/DDR3_A6 -> /FPGA Memory/DDR3_A9
- IC1 pad C3: /FPGA Memory/DDR3_A12 -> /FPGA Memory/DDR3_A6
- IC1 pad C4: /FPGA Memory/DDR3_A1 -> /FPGA Memory/DDR3_A8
- IC1 pad C5: /FPGA Memory/DDR3_A8 -> /FPGA Memory/DDR3_A5
- IC1 pad D1: /FPGA Memory/DDR3_DQ13 -> /FPGA Memory/DDR3_DQ15
- IC1 pad D3: Net-(IC1-PadD3) -> /FPGA Memory/DDR3_A14
- IC1 pad D5: /FPGA Memory/DDR3_A10 -> /FPGA Memory/DDR3_A11
- IC1 pad E1: /FPGA Memory/DDR3_DQ11 -> /FPGA Memory/DDR3_DQ9
- IC1 pad E2: /FPGA Memory/DDR3_DQ15 -> /FPGA Memory/DDR3_DQ13
- IC1 pad E3: /FPGA Memory/DDR3_A9 -> /FPGA Memory/DDR3_A15
- IC1 pad E4: /FPGA Memory/DDR3_A7 -> /FPGA Memory/DDR3_A12
- IC1 pad E5: /FPGA Memory/DDR3_A2 -> /FPGA Memory/DDR3_A1
- IC1 pad F2: Net-(IC1-PadF2) -> /FPGA Memory/DDR3_DQ11
- IC1 pad F3: /FPGA Memory/DDR3_DQ9 -> /FPGA Memory/~DDR3_CS
- IC1 pad F4: /FPGA Memory/DDR3_A5 -> /FPGA Memory/DDR3_A4
- IC1 pad F5: /FPGA Memory/DDR3_A3 -> /FPGA Memory/DDR3_A13
- IC1 pad G3: Net-(IC1-PadG3) -> /FPGA Memory/DDR3_A10
- IC1 pad J4: /FPGA Memory/DDR3_DM0 -> Net-(IC1-PadJ4)
- IC1 pad K4: /FPGA Memory/~DDR3_CS -> Net-(IC1-PadK4)
- IC1 pad L1: /FPGA Memory/~DDR3_CAS -> /FPGA Memory/~DDR3_RAS
- IC1 pad L4: Net-(IC1-PadL4) -> /FPGA Memory/DDR3_DM0
- IC1 pad M1: /FPGA Memory/~DDR3_WE -> /FPGA Memory/~DDR3_CAS
- IC1 pad M3: /FPGA Memory/DDR3_BA2 -> /FPGA Memory/~DDR3_WE
- IC1 pad N1: Net-(IC1-PadN1) -> /FPGA Memory/DDR3_BA2
- IC1 pad P1: /FPGA Memory/~DDR3_RAS -> Net-(IC1-PadP1)
- IC1 pad P2: /FPGA Memory/DDR3_A0 -> Net-(IC1-PadP2)
- IC1 pad P5: /FPGA Memory/DDR3_BA0 -> Net-(IC1-PadP5)
Routing:
- net /FPGA Memory/DDR3_A13: track 11.5 -> 41.5 mm, vias 2 -> 3
- net /FPGA Memory/DDR3_A8: track 11.5 -> 39.2 mm
- net /FPGA Memory/~DDR3_RAS: track 1.70 -> 28.8 mm, vias 2 -> 4
- net /FPGA Memory/DDR3_CKE: track 0.00 -> 26.4 mm, vias 0 -> 3
- net /FPGA Memory/DDR3_A9: track 11.5 -> 37.1 mm, vias 2 -> 3
- net /FPGA Memory/DDR3_A4: track 11.6 -> 36.4 mm
- net /FPGA Memory/DDR3_A6: track 11.6 -> 35.6 mm
- net /FPGA Memory/DDR3_A5: track 12.1 -> 35.8 mm
- net /FPGA Memory/DDR3_A2: track 12.0 -> 35.1 mm
- net /FPGA Memory/DDR3_A11: track 11.5 -> 34.3 mm, vias 2 -> 3
- net /FPGA Memory/DDR3_A1: track 11.5 -> 34.0 mm, vias 2 -> 3
- net /FPGA Memory/DDR3_A7: track 12.9 -> 35.1 mm
- net /FPGA Memory/DDR3_A14: track 11.5 -> 32.7 mm, vias 2 -> 3
- net /FPGA Memory/DDR3_A0: track 11.5 -> 32.4 mm, vias 2 -> 3
- net /FPGA Memory/~DDR3_WE: track 11.5 -> 32.1 mm, vias 2 -> 3
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Other:
- net class DDR3_CTRL: trace_width 0.14 -> 0.135
- net class DDR3_DQS: trace_width 0.1 -> 0.14

Commit message: More routing progress on Ethernet and DDR.
Parts:
- added H5: MountingHole, KiCAD_Magic:Keystone-4881, F.Cu at (165.8, 89.0)
- added R9: 47, Resistor_SMD:R_0402_1005Metric, B.Cu at (133.3, 85.5)
- added RN12: 47, Resistor_SMD:R_Array_Concave_4x0402, B.Cu at (147.9, 83.8)
- added RN9: 470, Resistor_SMD:R_Array_Concave_4x0603, F.Cu at (107.5, 53.2)
- C110, C111, C112, C113, C114, C115: footprint Capacitor_SMD:C_0603_1608Metric -> Capacitor_SMD:C_0402_1005Metric
- C401, C402, C404, C405, C406, C411, C413, C414, C415, C416, C421, C422, C423, C424, C425, C426, C430, C431, C433, C434, C435, C436, C462, C463, C464, C469, R3, R4: moved to B.Cu
- C460: moved to F.Cu
- RN1, RN2, RN3: footprint Resistor_THT:R_Array_SIP9 -> KiCAD_Magic:EXBD-1206; moved to B.Cu
- moved R3 324.1 mm to (152.2, 86.3)
- moved RN1 323.1 mm to (149.1, 86.7), turned to 90 degrees
- moved RN2 323.0 mm to (149.1, 90.7), turned to 270 degrees
- moved RN3 319.9 mm to (145.1, 87.5), turned to 90 degrees
- moved R4 308.7 mm to (142.1, 86.3)
- moved R7 303.4 mm to (121.5, 55.8), turned to 270 degrees
- moved C469 302.1 mm to (148.4, 81.7), turned to 90 degrees
- moved SW1 284.1 mm to (107.5, 57.8)
- moved C113 283.9 mm to (153.4, 59.5)
- moved C111 280.0 mm to (153.4, 57.5)
- moved C430 279.0 mm to (158.4, 105.8), turned to 90 degrees
- moved C115 278.1 mm to (153.4, 63.4)
- moved C112 276.4 mm to (153.4, 58.5)
- moved C431 275.6 mm to (152.4, 81.5), turned to 270 degrees
- moved C421 272.7 mm to (152.2, 85.1)
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Connections:
- IC1 pad A12: Net-(IC1-PadA12) -> /Ethernet/ETH_TXD0
- IC1 pad A13: Net-(IC1-PadA13) -> /Ethernet/ETH_TXD2
- IC1 pad A14: /Ethernet/MMC_CLK -> /Ethernet/LED_USER2
- IC1 pad A15: /Ethernet/MDIO_DATA -> /Ethernet/ETH_TXCLK
- IC1 pad A16: /Ethernet/ETH_TXD0 -> /Ethernet/ETH_RXD3
- IC1 pad A17: /Ethernet/ETH_RXD2 -> /Ethernet/ETH_RXD1
- IC1 pad A18: /Ethernet/ETH_TXCLK -> /Ethernet/ETH_RXCTL
- IC1 pad A19: /Ethernet/ETH_RXCLK -> /Ethernet/MDIO_CLK
- IC1 pad A3: /FPGA Memory/DDR3_A3 -> /FPGA Memory/DDR3_A8
- IC1 pad B12: /Ethernet/LED_USER3 -> /Ethernet/LED_USER4
- IC1 pad B13: Net-(IC1-PadB13) -> /Ethernet/ETH_TXD1
- IC1 pad B15: /Ethernet/MDIO_CLK -> Net-(IC1-PadB15)
- IC1 pad B16: /Ethernet/ETH_TXD1 -> /Ethernet/ETH_RXD2
- IC1 pad B17: /Ethernet/ETH_RXD0 -> /Ethernet/ETH_RXCLK
- IC1 pad B18: /Ethernet/ETH_RXD3 -> /Ethernet/ETH_RXD0
- IC1 pad B19: /Ethernet/ETH_RXCTL -> /Ethernet/MDIO_DATA
- IC1 pad B20: /Ethernet/ETH_TXCTL -> /Ethernet/~ETH_INT
- IC1 pad C1: /FPGA Memory/DDR3_DQ14 -> /FPGA Memory/DDR3_DQ12
- IC1 pad C12: /Ethernet/LED_USER4 -> /Ethernet/LED_USER3
- IC1 pad C13: /Ethernet/MMC_DAT2 -> /Ethernet/ETH_TXD3
- IC1 pad C14: /Ethernet/MMC_DAT0 -> /Ethernet/LED_USER1
- IC1 pad C15: /Ethernet/~ETH_RESET -> Net-(IC1-PadC15)
- IC1 pad C16: /Ethernet/ETH_TXD2 -> /Ethernet/ETH_TXCTL
- IC1 pad C17: /Ethernet/ETH_RXD1 -> /Ethernet/~ETH_RESET
- IC1 pad C18: /Exp Headers/P8_LVDS1p -> /Exp Headers/P8_LVDS7p
- IC1 pad C2: /FPGA Memory/DDR3_DQ12 -> /FPGA Memory/DDR3_DQ14
- IC1 pad C20: /Exp Headers/P8_LVDS9p -> /Exp Headers/P8_LVDS1p
- IC1 pad C3: /FPGA Memory/DDR3_A6 -> /FPGA Memory/DDR3_ODT1
- IC1 pad C4: /FPGA Memory/DDR3_A8 -> /FPGA Memory/DDR3_A6
- IC1 pad D11: /Ethernet/LED_USER1 -> Net-(IC1-PadD11)
- IC1 pad D13: /Ethernet/MMC_DAT3 -> /Ethernet/MMC_CLK
- IC1 pad D15: /Ethernet/~ETH_INT -> /Ethernet/MMC_DAT2
- IC1 pad D16: /Ethernet/ETH_TXD3 -> Net-(IC1-PadD16)
- IC1 pad D17: /Exp Headers/P8_LVDS1n -> /Exp Headers/P8_LVDS7n
- IC1 pad D18: /Exp Headers/P8_LVDS3p -> /Exp Headers/P8_LVDS8p
- IC1 pad D19: /Exp Headers/P8_LVDS9n -> /Exp Headers/P8_LVDS1n
- IC1 pad D2: Net-(IC1-PadD2) -> /FPGA Memory/~DDR3_WE
- IC1 pad D20: /Exp Headers/P8_LVDS10p -> /Exp Headers/P8_LVDS2p
- IC1 pad E11: /Ethernet/LED_USER2 -> /Ethernet/MMC_CMD
- IC1 pad E13: /Ethernet/MMC_CMD -> /Ethernet/MMC_DAT0
- IC1 pad E15: Net-(IC1-PadE15) -> /Ethernet/MMC_DAT3
- IC1 pad E16: /Exp Headers/P8_LVDS2p -> /Exp Headers/P8_LVDS11p
- IC1 pad E17: /Exp Headers/P8_LVDS3n -> /Exp Headers/P8_LVDS8n
- IC1 pad E18: /Exp Headers/P8_LVDS4p -> /Exp Headers/P8_LVDS9p
- IC1 pad E19: /Exp Headers/P8_LVDS10n -> /Exp Headers/P8_LVDS2n
- IC1 pad E20: /Exp Headers/P8_LVDS11p -> /Exp Headers/P8_LVDS3p
- IC1 pad F1: /FPGA Memory/DDR3_DQ6 -> /FPGA Memory/DDR3_DQ2
- IC1 pad F16: /Exp Headers/P8_LVDS2n -> /Exp Headers/P8_LVDS11n
- IC1 pad F17: /Exp Headers/P8_LVDS5p -> /Exp Headers/P8_LVDS10p
- IC1 pad F18: /Exp Headers/P8_LVDS4n -> /Exp Headers/P8_LVDS9n
- IC1 pad F19: /Exp Headers/P8_LVDS11n -> /Exp Headers/P8_LVDS3n
- IC1 pad F20: /Exp Headers/P8_LVDS12p -> /Exp Headers/P8_LVDS4p
- IC1 pad F3: /FPGA Memory/~DDR3_CS -> /FPGA Memory/DDR3_A3
- IC1 pad G1: /FPGA Memory/DDR3_DQ2 -> /FPGA Memory/DDR3_DQ6
- IC1 pad G16: /Exp Headers/P8_LVDS6p -> /Exp Headers/P8_LVDS12p
- IC1 pad G18: /Exp Headers/P8_LVDS5n -> /Exp Headers/P8_LVDS10n
- IC1 pad G19: /Exp Headers/P8_LVDS13p -> /Exp Headers/P8_LVDS5p
- IC1 pad G20: /Exp Headers/P8_LVDS12n -> /Exp Headers/P8_LVDS4n
- IC1 pad H16: /Exp Headers/P8_LVDS6n -> /Exp Headers/P8_LVDS12n
- IC1 pad H17: /Exp Headers/P8_LVDS7n -> /Exp Headers/P8_LVDS14n
- IC1 pad H18: /Exp Headers/P8_LVDS7p -> /Exp Headers/P8_LVDS14p
- IC1 pad H20: /Exp Headers/P8_LVDS13n -> /Exp Headers/P8_LVDS5n
- IC1 pad H5: /FPGA Memory/DDR3_DM1 -> /FPGA Memory/DDR3_BA1
- IC1 pad J16: /Exp Headers/P8_LVDS8n -> /Exp Headers/P8_LVDS13n
- IC1 pad J17: /Exp Headers/P8_LVDS8p -> /Exp Headers/P8_LVDS13p
- IC1 pad J18: /Exp Headers/P8_LVDS14p -> /Exp Headers/P8_LVDS16p
- IC1 pad J20: /Exp Headers/P8_LVDS16p -> /Exp Headers/P8_LVDS6p
- IC1 pad J5: Net-(IC1-PadJ5) -> /FPGA Memory/DDR3_DM1
- IC1 pad K18: /Exp Headers/P8_LVDS14n -> /Exp Headers/P8_LVDS16n
- IC1 pad K20: /Exp Headers/P8_LVDS16n -> /Exp Headers/P8_LVDS6n
- IC1 pad K4: Net-(IC1-PadK4) -> /FPGA Memory/DDR3_CKE
- IC1 pad L2: /FPGA Memory/DDR3_ODT0 -> Net-(IC1-PadL2)
- IC1 pad M1: /FPGA Memory/~DDR3_CAS -> /FPGA Memory/DDR3_BA2
- IC1 pad M3: /FPGA Memory/~DDR3_WE -> /FPGA Memory/~DDR3_CS
- IC1 pad N1: /FPGA Memory/DDR3_BA2 -> Net-(IC1-PadN1)
- IC1 pad N2: /FPGA Memory/DDR3_CKE -> /FPGA Memory/~DDR3_CAS
- IC1 pad N3: /FPGA Memory/DDR3_BA1 -> /FPGA Memory/DDR3_ODT0
- RN1 pad 2: /FPGA Memory/DDR3_BA0 -> /FPGA Memory/DDR3_BA1
- RN1 pad 3: /FPGA Memory/DDR3_BA1 -> /FPGA Memory/DDR3_A12
- RN1 pad 4: /FPGA Memory/DDR3_BA2 -> /FPGA Memory/DDR3_A10
- RN1 pad 5: /FPGA Memory/~DDR3_RAS -> /FPGA Memory/DDR3_CKE
- RN1 pad 6: /FPGA Memory/~DDR3_CAS -> /FPGA Memory/~DDR3_RAS
- RN1 pad 7: /FPGA Memory/~DDR3_CS -> /FPGA Memory/~DDR3_WE
- RN1 pad 8: /FPGA Memory/~DDR3_WE -> /FPGA Memory/DDR3_A15
- RN1 pad 9: /FPGA Memory/DDR3_CKE -> /FPGA Memory/DDR3_A2
- RN2 pad 2: /FPGA Memory/DDR3_A0 -> /FPGA Memory/DDR3_A1
- RN2 pad 3: /FPGA Memory/DDR3_A1 -> /FPGA Memory/DDR3_A11
- RN2 pad 4: /FPGA Memory/DDR3_A2 -> /FPGA Memory/DDR3_A9
- RN2 pad 5: /FPGA Memory/DDR3_A3 -> /FPGA Memory/DDR3_A13
- RN2 pad 6: /FPGA Memory/DDR3_A4 -> /FPGA Memory/DDR3_A8
- RN2 pad 7: /FPGA Memory/DDR3_A5 -> /FPGA Memory/DDR3_A14
- RN2 pad 8: /FPGA Memory/DDR3_A6 -> /FPGA Memory/DDR3_A4
- RN2 pad 9: /FPGA Memory/DDR3_A7 -> /FPGA Memory/DDR3_A6
- RN3 pad 2: /FPGA Memory/DDR3_A8 -> /FPGA Memory/DDR3_A5
- RN3 pad 3: /FPGA Memory/DDR3_A9 -> /FPGA Memory/DDR3_A0
- RN3 pad 4: /FPGA Memory/DDR3_A10 -> /FPGA Memory/DDR3_BA2
- RN3 pad 5: /FPGA Memory/DDR3_A11 -> /FPGA Memory/~DDR3_CAS
- RN3 pad 6: /FPGA Memory/DDR3_A12 -> /FPGA Memory/~DDR3_CS
- RN3 pad 7: /FPGA Memory/DDR3_A13 -> /FPGA Memory/DDR3_BA0
- RN3 pad 8: /FPGA Memory/DDR3_A14 -> /FPGA Memory/DDR3_A3
- RN3 pad 9: /FPGA Memory/DDR3_A15 -> /FPGA Memory/DDR3_A7
Routing:
- net GND: track 106.9 -> 209.4 mm, vias 47 -> 68
- net /Ethernet/MMC_DAT3: track 0.00 -> 44.3 mm, vias 0 -> 2
- net /Ethernet/MMC_DAT2: track 0.00 -> 43.1 mm, vias 0 -> 2
- net /Exp Headers/P8_LVDS16n: track 0.00 -> 41.6 mm, vias 0 -> 1
- net /Ethernet/MMC_CLK: track 0.00 -> 40.7 mm, vias 0 -> 2
- net /Exp Headers/P8_LVDS16p: track 0.00 -> 40.6 mm, vias 0 -> 1
- net /Exp Headers/P8_LVDS14n: track 0.00 -> 39.8 mm, vias 0 -> 1
- net /Ethernet/MMC_DAT1: track 0.00 -> 39.6 mm, vias 0 -> 2
- net /Exp Headers/P8_LVDS15n: track 0.00 -> 39.3 mm, vias 0 -> 1
- net /Ethernet/MMC_CMD: track 0.00 -> 39.3 mm, vias 0 -> 2
- net /Ethernet/MMC_DAT0: track 0.00 -> 38.9 mm, vias 0 -> 2
- net /Ethernet/MMC_DET: track 0.00 -> 38.7 mm, vias 0 -> 2
- net /Exp Headers/P8_LVDS13n: track 0.00 -> 38.2 mm, vias 0 -> 1
- net /Exp Headers/P8_LVDS15p: track 0.00 -> 37.5 mm, vias 0 -> 1
- net /Exp Headers/P8_LVDS12n: track 0.00 -> 36.6 mm, vias 0 -> 1
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- added copper zone on Gnd1.Cu, net GND
- added copper zone on Gnd3.Cu, net GND
Other:
- net class Default: trace_width 0.1 -> 0.135

Commit message: Routing of M.2 and PCIe, placed the Supervisor.
Started work on getting the power supplies layed out too, and spent
some time thinking about how the USB-C should connect up to the FPGA.
Parts:
- added C119: 1uF, Capacitor_SMD:C_0603_1608Metric, F.Cu at (111.0, 83.0)
- added D1: LED_ARGB, KiCAD_Magic:LTST-C19HE1WT, F.Cu at (107.5, 96.8)
- added D7: LED_ALT, LED_SMD:LED_0603_1608Metric, F.Cu at (182.2, 58.0)
- added D8: LED_ALT, LED_SMD:LED_0603_1608Metric, F.Cu at (182.2, 60.0)
- added IC15: TC7USB40MU, Package_DFN_QFN:UQFN-10_1.4x1.8mm_P0.4mm, F.Cu at (110.8, 87.5)
- added IC16: NCP349, Logicbone:DFN6_1.6x2mm, F.Cu at (110.7, 84.8)
- added IC7: FUSB302-QFN14, Package_DFN_QFN:WQFN-14-1EP_2.5x2.5mm_P0.5mm_EP1.45x1.45mm, F.Cu at (110.0, 91.5)
- added J5: Conn_02x05_Odd_Even, KiCAD_Magic:ftsh-105-01-dv, F.Cu at (177.2, 84.5)
- added R11: 10k, Resistor_SMD:R_0402_1005Metric, B.Cu at (179.2, 58.0)
- added R12: 10k, Resistor_SMD:R_0402_1005Metric, B.Cu at (179.2, 60.0)
- added R26: 1.5k, Resistor_SMD:R_0402_1005Metric, B.Cu at (135.7, 60.5)
- added RN10: 4.7k, Resistor_SMD:R_Array_Concave_4x0603, F.Cu at (169.5, 82.0)
- added RN11: 4.7k, Resistor_SMD:R_Array_Concave_4x0603, F.Cu at (169.5, 76.5)
- added RN4: 4.7k, Resistor_SMD:R_Array_Concave_4x0603, F.Cu at (76.0, 67.5)
- added RN5: 4.7k, Resistor_SMD:R_Array_Concave_4x0603, B.Cu at (67.5, 80.7)
- added RN6: 470, Resistor_SMD:R_Array_Concave_4x0603, F.Cu at (114.6, 91.5)
- added RN7: 4.7k, Resistor_SMD:R_Array_Concave_4x0603, F.Cu at (70.6, 80.7)
- added RN8: 4.7k, Resistor_SMD:R_Array_Concave_4x0603, B.Cu at (76.0, 87.0)
- C110, C111, C112, C113, C114, C115, C116, C118, C300, C301, C302, C305, C306, C307, C308, C309, C310, C311, C312, C313, C314, C315, C316, C317, C318, C319, FB6, FB7, R5: moved to B.Cu
- IC10: value AT25SF081-XMHF-X -> W25Q128JVSIQ; footprint Package_SO:TSSOP-8_4.4x3mm_P0.65mm -> Package_DFN_QFN:DFN-8-1EP_6x5mm_P1.27mm_EP2x2mm
- IC11: value FAN53600AUC33X -> FAN5362UMP; footprint Package_CSP:WLCSP-6_1.4x1.0mm_P0.4mm -> Package_DFN_QFN:DFN-6-1EP_2x2mm_P0.65mm_EP1x1.6mm
- J4: footprint KiCAD_Magic:ftsh-105-01-dv -> Connector:Tag-Connect_TC2050-IDC-NL_2x05_P1.27mm_Vertical
- moved C118 323.7 mm to (158.2, 88.7), turned to 180 degrees
- moved C116 317.7 mm to (157.3, 87.4)
- moved IC9 299.6 mm to (157.8, 89.0)
- moved R8 294.2 mm to (175.6, 70.5), turned to 270 degrees
- moved C109 289.2 mm to (175.6, 74.0), turned to 90 degrees
- moved C108 288.2 mm to (180.6, 74.0), turned to 270 degrees
- moved Y1 282.6 mm to (178.1, 74.0), turned to 180 degrees
- moved R5 273.8 mm to (151.4, 57.3), turned to 90 degrees
- moved R29 254.9 mm to (111.5, 57.8), turned to 90 degrees
- moved IC10 221.0 mm to (169.5, 71.2), turned to 180 degrees
- moved IC6 210.2 mm to (165.0, 81.2), turned to 90 degrees
- moved C305 201.2 mm to (127.8, 53.5), turned to 90 degrees
- moved J4 200.9 mm to (157.1, 67.0)
- moved C309 200.8 mm to (128.8, 56.5), turned to 270 degrees
- moved C313 196.7 mm to (129.8, 62.0), turned to 180 degrees
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Connections:
- net /FPGA SERDES/PCIE_RX0n renamed /FPGA SERDES/PCIE_RX0-
- net /FPGA SERDES/PCIE_RX0p renamed /FPGA SERDES/PCIE_RX0+
- net /FPGA SERDES/PCIE_RX1n renamed /FPGA SERDES/PCIE_RX1-
- net /FPGA SERDES/PCIE_RX1p renamed /FPGA SERDES/PCIE_RX1+
- net /FPGA SERDES/PCIE_TX0n renamed /FPGA SERDES/PCIE_TX0-
- net /FPGA SERDES/PCIE_TX0p renamed /FPGA SERDES/PCIE_TX0+
- net /FPGA SERDES/PCIE_TX1n renamed /FPGA SERDES/PCIE_TX1-
- net /FPGA SERDES/PCIE_TX1p renamed /FPGA SERDES/PCIE_TX1+
- C110 pad 2: /FPGA SERDES/SERDES_REFCLKn -> /FPGA SERDES/SERDES_REFCLK-
- C111 pad 2: /FPGA SERDES/SERDES_REFCLKp -> /FPGA SERDES/SERDES_REFCLK+
- IC1 pad A10: /Exp Headers/ADC_SCLK -> /Exp Headers/P9_GPIO13
- IC1 pad A11: /Exp Headers/ADC_MISO -> /Exp Headers/P9_GPIO11
- IC1 pad A13: /Ethernet/ETH_TXD2 -> /Ethernet/ETH_TXD1
- IC1 pad A14: /Ethernet/LED_USER2 -> /Ethernet/ETH_TXD3
- IC1 pad A15: /Ethernet/ETH_TXCLK -> /Ethernet/ETH_TXCTL
- IC1 pad A16: /Ethernet/ETH_RXD3 -> /Ethernet/ETH_RXD2
- IC1 pad A17: /Ethernet/ETH_RXD1 -> /Ethernet/ETH_RXD0
- IC1 pad A18: /Ethernet/ETH_RXCTL -> /Ethernet/ETH_RXCLK
- IC1 pad A6: /Exp Headers/P9_GPIO11 -> /Exp Headers/P9_GPIO25
- IC1 pad A7: /Exp Headers/P9_GPIO25 -> /Exp Headers/P9_GPIO24
- IC1 pad A8: /Exp Headers/P9_GPIO26 -> /Exp Headers/P9_GPIO18
- IC1 pad A9: /Exp Headers/P9_CLKOUT -> /Exp Headers/P9_GPIO15
- IC1 pad B10: /Exp Headers/~ADC_CSEL -> /Exp Headers/P9_CLKOUT
- IC1 pad B11: /Exp Headers/ADC_MOSI -> /Exp Headers/P9_GPIO12
- IC1 pad B12: /Ethernet/LED_USER4 -> /Ethernet/FPGA_USB+
- IC1 pad B13: /Ethernet/ETH_TXD1 -> /Ethernet/LED_USER4
- IC1 pad B15: Net-(IC1-PadB15) -> /Ethernet/ETH_TXCLK
- IC1 pad B16: /Ethernet/ETH_RXD2 -> /Ethernet/ETH_RXD3
- IC1 pad B17: /Ethernet/ETH_RXCLK -> /Ethernet/ETH_RXD1
- IC1 pad B18: /Ethernet/ETH_RXD0 -> /Ethernet/ETH_RXCTL
- IC1 pad B6: /Exp Headers/P9_GPIO12 -> /Exp Headers/P9_GPIO26
- IC1 pad B8: /Exp Headers/P9_GPIO24 -> /Exp Headers/P9_GPIO23
- IC1 pad B9: /Exp Headers/P9_SPI_D0 -> /Exp Headers/P9_GPIO16
- IC1 pad C10: Net-(IC1-PadC10) -> /Exp Headers/P9_GPIO14
- IC1 pad C11: Net-(IC1-PadC11) -> /Exp Headers/P9_GPIO17
- IC1 pad C12: /Ethernet/LED_USER3 -> /Ethernet/FPGA_USB-
- IC1 pad C13: /Ethernet/ETH_TXD3 -> /Ethernet/LED_USER3
- IC1 pad C14: /Ethernet/LED_USER1 -> /Ethernet/ETH_TXD2
- IC1 pad C15: Net-(IC1-PadC15) -> /Ethernet/LED_USER2
- IC1 pad C16: /Ethernet/ETH_TXCTL -> /Ethernet/FPGA_USB_PULL
- IC1 pad C6: /Exp Headers/P9_GPIO17 -> /Exp Headers/P9_SPI_D1
- IC1 pad C7: /Exp Headers/P9_GPIO18 -> /Exp Headers/~P9_SPI_CSEL
- IC1 pad C8: /Exp Headers/P9_GPIO23 -> /Exp Headers/P9_GPIO22
- IC1 pad C9: /Exp Headers/~P9_SPI_CSEL -> Net-(IC1-PadC9)
- IC1 pad D10: /Exp Headers/P9_SPI_SCLK -> /Exp Headers/P9_GPIO21
- IC1 pad D13: /Ethernet/MMC_CLK -> /Ethernet/MMC_DAT0
- IC1 pad D15: /Ethernet/MMC_DAT2 -> /Ethernet/MMC_DAT3
- IC1 pad D16: Net-(IC1-PadD16) -> /Ethernet/LED_USER1
- IC1 pad D6: /Exp Headers/P9_GPIO14 -> /Exp Headers/P9_SPI_SCLK
- IC1 pad D7: /Exp Headers/P9_GPIO16 -> /Exp Headers/P9_SPI_D0
- IC1 pad D8: /Exp Headers/P9_GPIO22 -> /Exp Headers/P9_GPIO27
- IC1 pad D9: /Exp Headers/P9_GPIO27 -> /Exp Headers/ADC_SCLK
- IC1 pad E10: /Exp Headers/P9_SPI_D1 -> /Exp Headers/P9_GPIO42
- IC1 pad E11: /Ethernet/MMC_CMD -> /Ethernet/MMC_CLK
- IC1 pad E13: /Ethernet/MMC_DAT0 -> /Ethernet/MMC_DAT2
- IC1 pad E15: /Ethernet/MMC_DAT3 -> /Ethernet/MMC_CMD
- IC1 pad E6: /Exp Headers/P9_GPIO13 -> /Exp Headers/~ADC_CSEL
- IC1 pad E7: /Exp Headers/P9_GPIO15 -> Net-(IC1-PadE7)
- IC1 pad E8: /Exp Headers/P9_GPIO21 -> /Exp Headers/ADC_MOSI
- IC1 pad E9: /Exp Headers/P9_GPIO42 -> /Exp Headers/ADC_MISO
- IC1 pad L16: /FPGA SERDES/M2_SDIO_DATA2 -> /FPGA SERDES/~M2_WDIS2
- IC1 pad L17: /FPGA SERDES/M2_SDIO_DATA3 -> /FPGA SERDES/~PCIE_RESET0
- IC1 pad L18: /FPGA SERDES/~M2_SDIO_WAKE -> /FPGA SERDES/~PCIE_RESET1
- IC1 pad L19: /FPGA SERDES/M2_SDIO_DATA0 -> /FPGA SERDES/~M2_WDIS1
- IC1 pad L20: /FPGA SERDES/M2_SDIO_CLK -> /FPGA SERDES/~M2_SDIO_RESET
- IC1 pad M17: /FPGA SERDES/M2_PCM_SYNC -> /FPGA SERDES/~M2_ALERT
- IC1 pad M18: /FPGA SERDES/~M2_SDIO_RESET -> /FPGA SERDES/M2_SUSCLK
- IC1 pad M19: /FPGA SERDES/M2_SDIO_DATA1 -> /FPGA SERDES/~PCIE_WAKE0
- IC1 pad M20: /FPGA SERDES/M2_SDIO_CMD -> /FPGA SERDES/~PCIE_WAKE1
- IC1 pad N16: /FPGA SERDES/M2_PCM_CLK -> /FPGA SERDES/M2_PCM_SYNC
- IC1 pad N17: /FPGA SERDES/M2_RTS -> /FPGA SERDES/M2_SDIO_CLK
- IC1 pad N18: /FPGA SERDES/M2_PCM_IN -> /FPGA SERDES/M2_VEND1
- IC1 pad N19: /FPGA SERDES/M2_COEX1 -> /FPGA SERDES/~M2_SDIO_WAKE
- IC1 pad N20: /FPGA SERDES/M2_COEX2 -> /FPGA SERDES/M2_COEX3
- IC1 pad P16: /FPGA SERDES/M2_CTS -> /FPGA SERDES/M2_PCM_IN
- IC1 pad P17: /FPGA SERDES/M2_PCM_OUT -> /FPGA SERDES/M2_RTS
- IC1 pad P18: /FPGA SERDES/~M2_RESET -> /FPGA SERDES/M2_COEX2
- IC1 pad P19: /FPGA SERDES/M2_COEX3 -> /FPGA SERDES/M2_VEND2
- IC1 pad P20: /FPGA SERDES/~M2_WDIS1 -> /FPGA SERDES/M2_SDIO_DATA3
- IC1 pad P3: Net-(IC1-PadP3) -> /FPGA SERDES/FPGA_REFCLK+
- IC1 pad P4: Net-(IC1-PadP4) -> /FPGA SERDES/FPGA_REFCLK-
- IC1 pad R1: /Exp Headers/SCL -> /Exp Headers/SDA
- IC1 pad R18: /FPGA SERDES/M2_VEND1 -> /FPGA SERDES/M2_CTS
- IC1 pad R20: /FPGA SERDES/~M2_WDIS2 -> /FPGA SERDES/M2_SDIO_DATA2
- IC1 pad T1: /Exp Headers/SDA -> /Exp Headers/SCL
- IC1 pad T16: Net-(IC1-PadT16) -> /FPGA SERDES/M2_PCM_OUT
- IC1 pad T17: /FPGA SERDES/FPGA_REFCLKn -> /FPGA SERDES/M2_COEX1
- IC1 pad T18: /FPGA SERDES/~M2_ALERT -> /FPGA SERDES/~M2_UART_WAKE
- IC1 pad T19: /FPGA SERDES/M2_VEND2 -> /FPGA SERDES/M2_VEND0
- IC1 pad T20: /FPGA SERDES/~PCIE_WAKE0 -> /FPGA SERDES/M2_SDIO_DATA1
- IC1 pad U1: Net-(IC1-PadU1) -> /Supervisor/FPGA_UART_RXD
- IC1 pad U16: /FPGA SERDES/FPGA_REFCLKp -> /FPGA SERDES/M2_PCM_CLK
- IC1 pad U19: /FPGA SERDES/M2_VEND0 -> /FPGA SERDES/M2_SDIO_CMD
- IC1 pad U20: /FPGA SERDES/~PCIE_WAKE1 -> /FPGA SERDES/M2_SDIO_DATA0
- IC1 pad V1: /Supervisor/FPGA_UART_CLK -> /Supervisor/FPGA_UART_TXD
- IC1 pad W1: /Supervisor/FPGA_UART_TXD -> /Supervisor/FPGA_UART_CLK
- IC1 pad Y2: /Supervisor/FPGA_UART_RXD -> Net-(IC1-PadY2)
- IC10 pad 2: /Supervisor/FLASH_D0 -> /Supervisor/FLASH_D1
- IC4 pad 36: Net-(IC4-Pad36) -> /Supervisor/LED_BLUE
- IC4 pad 43: /Supervisor/LED_BLUE -> Net-(IC4-Pad43)
- IC5 pad 13: /FPGA SERDES/SERDES_REFCLKp -> /FPGA SERDES/FPGA_REFCLK+
- IC5 pad 14: /FPGA SERDES/SERDES_REFCLKn -> /FPGA SERDES/FPGA_REFCLK-
- IC5 pad 17: /FPGA SERDES/~PCIE_CLKREQ0 -> /FPGA SERDES/~PCIE_CLKREQ1
- IC5 pad 18: /FPGA SERDES/PCIE_REFCLK0p -> /FPGA SERDES/PCIE_REFCLK1-
- IC5 pad 19: /FPGA SERDES/PCIE_REFCLK0n -> /FPGA SERDES/PCIE_REFCLK1+
- IC5 pad 22: /FPGA SERDES/PCIE_REFCLK1p -> /FPGA SERDES/PCIE_REFCLK0-
- IC5 pad 23: /FPGA SERDES/PCIE_REFCLK1n -> /FPGA SERDES/PCIE_REFCLK0+
- IC5 pad 24: /FPGA SERDES/~PCIE_CLKREQ1 -> /FPGA SERDES/~PCIE_CLKREQ0
- IC5 pad 27: /FPGA SERDES/FPGA_REFCLKp -> /FPGA SERDES/SERDES_REFCLK-
- IC5 pad 28: /FPGA SERDES/FPGA_REFCLKn -> /FPGA SERDES/SERDES_REFCLK+
- IC6 pad 1: /Exp Headers/PWR_BUTTON -> /Ethernet/~SYS_RESET
- IC6 pad 2: /Ethernet/~SYS_RESET -> /Exp Headers/PWR_BUTTON
- IC8 pad 15: Net-(IC8-Pad15) -> /Supervisor/PMIC_VSELR2
- IC8 pad 20: /Exp Headers/PWR_BUTTON -> /Supervisor/FPGA_DONE
- IC8 pad 32: /Supervisor/USB_DM -> /Supervisor/STM_USB-
- IC8 pad 33: /Supervisor/USB_DP -> /Supervisor/STM_USB+
- IC8 pad 38: /Supervisor/PMIC_VSELR2 -> /Supervisor/~FPGA_HOLDN
- IC8 pad 45: /Ethernet/~SYS_RESET -> /Exp Headers/PWR_BUTTON
- IC8 pad 46: /Supervisor/FPGA_DONE -> /Ethernet/~SYS_RESET
- J1 pad 16: Net-(J1-Pad16) -> /FPGA SERDES/M2_LED2
- J1 pad 20: Net-(J1-Pad20) -> /FPGA SERDES/~M2_UART_WAKE
- J1 pad 47: /FPGA SERDES/PCIE_REFCLK0p -> /FPGA SERDES/PCIE_REFCLK0+
- J1 pad 49: /FPGA SERDES/PCIE_REFCLK0n -> /FPGA SERDES/PCIE_REFCLK0-
- J1 pad 50: Net-(J1-Pad50) -> /FPGA SERDES/M2_SUSCLK
- J1 pad 52: Net-(J1-Pad52) -> /FPGA SERDES/~PCIE_RESET0
- J1 pad 6: Net-(J1-Pad6) -> /FPGA SERDES/M2_LED1
- J1 pad 66: Net-(J1-Pad66) -> /FPGA SERDES/~PCIE_RESET1
- J1 pad 71: /FPGA SERDES/PCIE_REFCLK1p -> /FPGA SERDES/PCIE_REFCLK1+
- J1 pad 73: /FPGA SERDES/PCIE_REFCLK1n -> /FPGA SERDES/PCIE_REFCLK1-
- J2 pad A4: VBUS -> Net-(C119-Pad1)
- J2 pad A5: Net-(IC7-PadC1) -> /Supervisor/USB_CC1
- J2 pad A6: /Supervisor/USB_DP -> /Supervisor/USB_D+
- J2 pad A7: /Supervisor/USB_DM -> /Supervisor/USB_D-
- J2 pad A8: (no net) -> Net-(J2-PadA8)
- J2 pad A9: VBUS -> Net-(C119-Pad1)
- J2 pad B5: Net-(IC7-PadA1) -> /Supervisor/USB_CC2
- J2 pad B6: /Supervisor/USB_DP -> /Supervisor/USB_D+
- J2 pad B7: /Supervisor/USB_DM -> /Supervisor/USB_D-
- J2 pad B8: (no net) -> Net-(J2-PadB8)
- J4 pad 2: Net-(J4-Pad2) -> GND
- J4 pad 4: Net-(J4-Pad2) -> GND
- J4 pad 8: Net-(J4-Pad2) -> GND
- L12 pad 2: Net-(IC11-PadB1) -> Net-(IC11-Pad2)
Routing:
- net /Ethernet/~SYS_RESET: track 0.00 -> 161.0 mm, vias 0 -> 5
- net GND: track 209.4 -> 359.9 mm, vias 68 -> 114
- net /Exp Headers/SCL: track 0.00 -> 144.2 mm, vias 0 -> 5
- net /Exp Headers/SDA: track 0.00 -> 136.5 mm, vias 0 -> 5
- net /Supervisor/~USB_INT: track 0.00 -> 72.8 mm, vias 0 -> 2
- net /Supervisor/~PMIC_INT: track 0.00 -> 66.3 mm, vias 0 -> 2
- net /Ethernet/25M_REFCLK: track 1.06 -> 66.2 mm, vias 1 -> 2
- net /Exp Headers/P9_CLKOUT: track 0.00 -> 60.5 mm, vias 0 -> 1
- net /Supervisor/STM_USB+: track 0.00 -> 57.5 mm, vias 0 -> 1
- net /Supervisor/STM_USB-: track 0.00 -> 57.3 mm, vias 0 -> 1
- net /Exp Headers/P9_SPI_SCLK: track 0.00 -> 55.2 mm, vias 0 -> 1
- net /Exp Headers/P9_SPI_D0: track 0.00 -> 54.8 mm, vias 0 -> 1
- net /Exp Headers/P9_GPIO27: track 0.00 -> 54.7 mm, vias 0 -> 1
- net /Supervisor/PMIC_PWRHOLD: track 0.00 -> 54.3 mm, vias 0 -> 2
- net /Exp Headers/P9_GPIO42: track 0.57 -> 54.2 mm
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Other:
- net class PCIE added: clearance 0.08, trace_width 0.14, via_dia 0.5, via_drill 0.2
